File: universal-psu.kicad_pcb (KiCad board)
At the start: 0 parts

Commit message: Layout import and schema fixes.
Parts:
- added C1: 10u_50V_1210, Capacitor_SMD:C_1210_3225Metric, F.Cu at (162.8, -10.7)
- added C10: 47n_16V_0603, Capacitor_SMD:C_0201_0603Metric, F.Cu at (174.8, 11.1)
- added C11: 22u_25V_1210, Capacitor_SMD:C_1210_3225Metric, F.Cu at (174.1, -6.45)
- added C12: 1u_25V_1210, Capacitor_SMD:C_1210_3225Metric, F.Cu at (174.1, -2.20)
- added C13: 10u_50V_1210, Capacitor_SMD:C_1210_3225Metric, F.Cu at (119.8, 162.3)
- added C14: 10u_50V_1210, Capacitor_SMD:C_1210_3225Metric, F.Cu at (119.8, 166.6)
- added C15: 47n_16V_0603, Capacitor_SMD:C_0201_0603Metric, F.Cu at (131.8, 182.4)
- added C16: 100u_50V_1210, Capacitor_THT:CP_Radial_D4.0mm_P2.00mm, F.Cu at (126.9, 184.3)
- added C17: 22u_25V_1210, Capacitor_SMD:C_1210_3225Metric, F.Cu at (119.8, 170.8)
- added C18: 22u_25V_1210, Capacitor_SMD:C_1210_3225Metric, F.Cu at (125.4, 162.3)
- added C19: 2.2n_25V_1210, Capacitor_SMD:C_1210_3225Metric, F.Cu at (125.4, 166.6)
- added C2: 10u_50V_1210, Capacitor_SMD:C_1210_3225Metric, F.Cu at (162.8, -6.45)
- added C20: 1u_25V_1210, Capacitor_SMD:C_1210_3225Metric, F.Cu at (125.4, 170.8)
- added C21: 22u_25V_1210, Capacitor_SMD:C_1210_3225Metric, F.Cu at (131.1, 162.3)
- added C22: 47n_16V_0603, Capacitor_SMD:C_0201_0603Metric, F.Cu at (131.8, 184.2)
- added C23: 22u_25V_1210, Capacitor_SMD:C_1210_3225Metric, F.Cu at (131.1, 166.6)
- added C24: 1u_25V_1210, Capacitor_SMD:C_1210_3225Metric, F.Cu at (131.1, 170.8)
- added C3: 47n_16V_0603, Capacitor_SMD:C_0201_0603Metric, F.Cu at (174.8, 9.35)
- added C4: 100u_50V_1210, Capacitor_THT:CP_Radial_D4.0mm_P2.00mm, F.Cu at (169.9, 11.2)
- added C5: 22u_25V_1210, Capacitor_SMD:C_1210_3225Metric, F.Cu at (162.8, -2.20)
- added C6: 22u_25V_1210, Capacitor_SMD:C_1210_3225Metric, F.Cu at (168.4, -10.7)
- added C7: 2.2n_25V_1210, Capacitor_SMD:C_1210_3225Metric, F.Cu at (168.4, -6.45)
- added C8: 1u_25V_1210, Capacitor_SMD:C_1210_3225Metric, F.Cu at (168.4, -2.20)
- added C9: 22u_25V_1210, Capacitor_SMD:C_1210_3225Metric, F.Cu at (174.1, -10.7)
- added J1: Screw_Terminal_01x04, TerminalBlock_Phoenix:TerminalBlock_Phoenix_MKDS-1,5-4-5.08_1x04_P5.08mm_Horizontal, F.Cu at (25.2, 43.1)
- added J2: Screw_Terminal_01x04, TerminalBlock_Phoenix:TerminalBlock_Phoenix_MKDS-1,5-4-5.08_1x04_P5.08mm_Horizontal, F.Cu at (212.9, 75.5)
- added J3: Screw_Terminal_01x04, TerminalBlock_Phoenix:TerminalBlock_Phoenix_MKDS-1,5-4-5.08_1x04_P5.08mm_Horizontal, F.Cu at (212.3, 34.5)
- added PS1: IRM-60-15, Converter_ACDC:Converter_ACDC_MeanWell_IRM-60-xx_THT, F.Cu at (40.8, 30.2)
- added PS2: TLVM14406RCHR, footprints:CONV_TLVM14406RCHR, F.Cu at (173.2, 4.20)
- added PS3: TLVM14406RCHR, footprints:CONV_TLVM14406RCHR, F.Cu at (130.2, 177.2)
- added R1: 10k_0.21W_0603, Resistor_SMD:R_0603_1608Metric_Pad0.98x0.95mm_HandSolder, F.Cu at (157.8, -11.6)
- added R10: 0_0.21W_0603, Resistor_SMD:R_0603_1608Metric_Pad0.98x0.95mm_HandSolder, F.Cu at (157.8, 11.0)
- added R11: 10k_0.21W_0603, Resistor_SMD:R_0603_1608Metric_Pad0.98x0.95mm_HandSolder, F.Cu at (114.8, 161.5)
- added R12: 100_0.21W_0603, Resistor_SMD:R_0603_1608Metric_Pad0.98x0.95mm_HandSolder, F.Cu at (114.8, 164.0)
- added R13: 31.6k_0.21W_0603, Resistor_SMD:R_0603_1608Metric_Pad0.98x0.95mm_HandSolder, F.Cu at (114.8, 166.5)
- added R14: 10k_0.21W_0603, Resistor_SMD:R_0603_1608Metric_Pad0.98x0.95mm_HandSolder, F.Cu at (114.8, 169.0)
- added R15: 0_0.21W_0603, Resistor_SMD:R_0603_1608Metric_Pad0.98x0.95mm_HandSolder, F.Cu at (114.8, 171.5)
- added R16: 31.6k_0.21W_0603, Resistor_SMD:R_0603_1608Metric_Pad0.98x0.95mm_HandSolder, F.Cu at (114.8, 174.0)
- added R17: 9.53k_0.21W_0603, Resistor_SMD:R_0603_1608Metric_Pad0.98x0.95mm_HandSolder, F.Cu at (114.8, 176.5)
- added R18: 10k_0.21W_0603, Resistor_SMD:R_0603_1608Metric_Pad0.98x0.95mm_HandSolder, F.Cu at (114.8, 179.1)
- added R19: 11k_0.21W_0603, Resistor_SMD:R_0603_1608Metric_Pad0.98x0.95mm_HandSolder, F.Cu at (114.8, 181.6)
- added R2: 100_0.21W_0603, Resistor_SMD:R_0603_1608Metric_Pad0.98x0.95mm_HandSolder, F.Cu at (157.8, -9.06)
- added R20: 0_0.21W_0603, Resistor_SMD:R_0603_1608Metric_Pad0.98x0.95mm_HandSolder, F.Cu at (114.8, 184.1)
- added R3: 52.3k_0.21W_0603, Resistor_SMD:R_0603_1608Metric_Pad0.98x0.95mm_HandSolder, F.Cu at (157.8, -6.55)
- added R4: 10k_0.21W_0603, Resistor_SMD:R_0603_1608Metric_Pad0.98x0.95mm_HandSolder, F.Cu at (157.8, -4.04)
- added R5: 0_0.21W_0603, Resistor_SMD:R_0603_1608Metric_Pad0.98x0.95mm_HandSolder, F.Cu at (157.8, -1.53)
- added R6: 7.15k_0.21W_0603, Resistor_SMD:R_0603_1608Metric_Pad0.98x0.95mm_HandSolder, F.Cu at (157.8, 0.98)
- added R7: 9.53k_0.21W_0603, Resistor_SMD:R_0603_1608Metric_Pad0.98x0.95mm_HandSolder, F.Cu at (157.8, 3.49)
- added R8: 10k_0.21W_0603, Resistor_SMD:R_0603_1608Metric_Pad0.98x0.95mm_HandSolder, F.Cu at (157.8, 6.00)
- added R9: 11k_0.21W_0603, Resistor_SMD:R_0603_1608Metric_Pad0.98x0.95mm_HandSolder, F.Cu at (157.8, 8.51)
- added TP1: 12V, TestPoint:TestPoint_Pad_2.0x2.0mm, F.Cu at (161.9, 1.95)
- added TP10: FB, TestPoint:TestPoint_Pad_2.0x2.0mm, F.Cu at (119.0, 183.1)
- added TP11: GND, TestPoint:TestPoint_Pad_2.0x2.0mm, F.Cu at (119.0, 187.2)
- added TP12: RT, TestPoint:TestPoint_Pad_2.0x2.0mm, F.Cu at (123.0, 175.0)
- added TP13: GND, TestPoint:TestPoint_Pad_2.0x2.0mm, F.Cu at (123.0, 179.1)
- added TP14: 5V, TestPoint:TestPoint_Pad_2.0x2.0mm, F.Cu at (123.0, 183.1)
- added TP2: GND, TestPoint:TestPoint_Pad_2.0x2.0mm, F.Cu at (161.9, 6.00)
- added TP3: FB, TestPoint:TestPoint_Pad_2.0x2.0mm, F.Cu at (161.9, 10.1)
- added TP4: GND, TestPoint:TestPoint_Pad_2.0x2.0mm, F.Cu at (161.9, 14.1)
- added TP5: RT, TestPoint:TestPoint_Pad_2.0x2.0mm, F.Cu at (166.0, 1.95)
- added TP6: GND, TestPoint:TestPoint_Pad_2.0x2.0mm, F.Cu at (166.0, 6.00)
- added TP7: 5V, TestPoint:TestPoint_Pad_2.0x2.0mm, F.Cu at (166.0, 10.1)
- added TP8: 12V, TestPoint:TestPoint_Pad_2.0x2.0mm, F.Cu at (119.0, 175.0)
- added TP9: GND, TestPoint:TestPoint_Pad_2.0x2.0mm, F.Cu at (119.0, 179.1)
Other:
- copper layers 0 -> 2
