File: Subsheets/DC_DC_Converter_3v3.kicad_sch (KiCad schematic)
At the start: 30 parts

Commit message: Layout import and schema fixes.
Parts:
- C19: footprint (none) -> Capacitor_SMD:C_1210_3225Metric
- PS3: footprint TLVM14406RCHR:CONV_TLVM14406RCHR -> footprints:CONV_TLVM14406RCHR; Manufacturer Part Number (none) -> TLVM14406RCHR; Price (none) -> 742; Vendor Link (none) -> https://www.digikey.in/en/products/detail/texas-instruments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; Vendor Part Number (none) -> 296-TLVM14406RCHRCT-ND
- R11, R14, R18: footprint (none) -> Resistor_SMD:R_0603_1608Metric_Pad0.98x0.95mm_HandSolder; MANUFACTURER (none) -> Vishay Dale; Manufacturer Part Number (none) -> CRCW060310K0FKEAHP; Price (none) -> 6.01; Vendor Link (none) -> https://www.digikey.in/en/products/detail/vishay-dale/CRCW0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; Vendor Part Number (none) -> 541-10.0KSCT-ND
- R12: footprint (none) -> Resistor_SMD:R_0603_1608Metric_Pad0.98x0.95mm_HandSolder; MANUFACTURER (none) -> Vishay Dale; Manufacturer Part Number (none) -> CRCW0603100RFKEAHP; Price (none) -> 6.01; Vendor Link (none) -> https://www.digikey.in/en/products/detail/vishay-dale/CRCW0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; Vendor Part Number (none) -> 541-100SCT-ND
- R13: value 31.2k_0.21W_0603 -> 31.6k_0.21W_0603; footprint (none) -> Resistor_SMD:R_0603_1608Metric_Pad0.98x0.95mm_HandSolder; MANUFACTURER (none) -> Vishay Dale; Manufacturer Part Number (none) -> CRCW060331K6FKEAC; Price (none) -> 2.56; Vendor Link (none) -> https://www.digikey.in/en/products/detail/vishay-dale/CRCW0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; Vendor Part Number (none) -> 541-5351-1-ND
- R15, R20: footprint (none) -> Resistor_SMD:R_0603_1608Metric_Pad0.98x0.95mm_HandSolder; MANUFACTURER (none) -> Vishay Dale; Manufacturer Part Number (none) -> CRCW06030000Z0EAHP; Price (none) -> 4.86; Vendor Link (none) -> https://www.digikey.in/en/products/detail/vishay-dale/CRCW0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; Vendor Part Number (none) -> 541-0.0SBCT-ND
- R16: footprint (none) -> Resistor_SMD:R_0603_1608Metric_Pad0.98x0.95mm_HandSolder; MANUFACTURER (none) -> Vishay Dale; Manufacturer Part Number (none) -> CRCW060331K6FKEAC; Price (none) -> 2.56; Vendor Link (none) -> https://www.digikey.in/en/products/detail/vishay-dale/CRCW0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; Vendor Part Number (none) -> 541-5351-1-ND
- R17: footprint (none) -> Resistor_SMD:R_0603_1608Metric_Pad0.98x0.95mm_HandSolder; MANUFACTURER (none) -> Vishay Dale; Manufacturer Part Number (none) -> CRCW06039K53FKEAC; Price (none) -> 2.56; Vendor Link (none) -> https://www.digikey.in/en/products/detail/vishay-dale/CRCW0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; Vendor Part Number (none) -> 541-5606-1-ND
- R19: footprint (none) -> Resistor_SMD:R_0603_1608Metric_Pad0.98x0.95mm_HandSolder; MANUFACTURER (none) -> Vishay Dale; Manufacturer Part Number (none) -> CRCW060311K0FKEAC; Price (none) -> 2.56; Vendor Link (none) -> https://www.digikey.in/en/products/detail/vishay-dale/CRCW0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; Vendor Part Number (none) -> 541-5146-1-ND
- TP10, TP11, TP12, TP13, TP14, TP8, TP9: footprint (none) -> TestPoint:TestPoint_Pad_2.0x2.0mm

Commit message: layout changes
Parts:
- renumbered TP8 to 12V, TP14 to 3v3, TP10 to 3v3_FB, TP12 to 3v3_RT, TP13 to GND, TP9 to GND, TP11 to GND
Changed lines of the file:
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@@
 		(on_board yes)
 		(dnp no)
-		(property "Reference" "TP14"
+		(property "Reference" "3v3"
 			(at 86.106 151.13 0)
 			(show_name no)
@@
 			(project "universal-psu"
 				(path "/08cd4a39-b122-4f15-a276-9889e34f331e/fea1cda1-5d74-450c-bf04-495c5d5714c3"
-					(reference "TP14")
+					(reference "3v3")
 					(unit 1)
 				)
@@
 		(on_board yes)
 		(dnp no)
-		(property "Reference" "TP10"
+		(property "Reference" "3v3_FB"
 			(at 62.992 151.13 0)
 			(show_name no)
@@
 			(project "universal-psu"
 				(path "/08cd4a39-b122-4f15-a276-9889e34f331e/fea1cda1-5d74-450c-bf04-495c5d5714c3"
-					(reference "TP10")
+					(reference "3v3_FB")
 					(unit 1)
 				)
@@
 		(on_board yes)
 		(dnp no)
-		(property "Reference" "TP12"
+		(property "Reference" "3v3_RT"
 			(at 73.152 151.13 0)
 			(show_name no)
@@
 			(project "universal-psu"
 				(path "/08cd4a39-b122-4f15-a276-9889e34f331e/fea1cda1-5d74-450c-bf04-495c5d5714c3"
-					(reference "TP12")
+					(reference "3v3_RT")
 					(unit 1)
 				)
@@
 		(on_board yes)
 		(dnp no)
-		(property "Reference" "TP8"
+		(property "Reference" "12V"
 			(at 51.816 151.13 0)
 			(show_name no)
@@
 			(project "universal-psu"
 				(path "/08cd4a39-b122-4f15-a276-9889e34f331e/fea1cda1-5d74-450c-bf04-495c5d5714c3"
-					(reference "TP8")
+					(reference "12V")
 					(unit 1)
 				)
@@
 		(on_board yes)
 		(dnp no)
-		(property "Reference" "TP13"
+		(property "Reference" "GND"
 			(at 73.152 161.29 0)
 			(show_name no)
@@
 			(project "universal-psu"
 				(path "/08cd4a39-b122-4f15-a276-9889e34f331e/fea1cda1-5d74-450c-bf04-495c5d5714c3"
-					(reference "TP13")
+					(reference "GND")
 					(unit 1)
 				)
@@
 		(on_board yes)
 		(dnp no)
-		(property "Reference" "TP9"
+		(property "Reference" "GND"
 			(at 57.912 161.29 0)
 			(show_name no)
@@
 			(project "universal-psu"
 				(path "/08cd4a39-b122-4f15-a276-9889e34f331e/fea1cda1-5d74-450c-bf04-495c5d5714c3"
-					(reference "TP9")
+					(reference "GND")
 					(unit 1)
 				)
@@
 		(on_board yes)
 		(dnp no)
-		(property "Reference" "TP11"
+		(property "Reference" "GND"
 			(at 65.532 161.29 0)
 			(show_name no)
@@
 			(project "universal-psu"
 				(path "/08cd4a39-b122-4f15-a276-9889e34f331e/fea1cda1-5d74-450c-bf04-495c5d5714c3"
-					(reference "TP11")
+					(reference "GND")
 					(unit 1)
 				)

Commit message: Layout  closed, some DRC  conflicts remain.
Parts:
- added R22: 10k_0.21W_0603, Resistor_SMD:R_0603_1608Metric_Pad0.98x0.95mm_HandSolder, symbol Device:R
- renumbered 12V to 12V2, 3v3_FB to 3v3_FB1, 3v3_RT to 3v3_RT1, GND to GND4, GND to GND5, GND to GND6
Connections:
- net GND: now also R22.2
- net PG: now also R22.1
Other:
- moved on the sheet: C19, C22, R19
