File: Subsheets/DC_DC_Converter_5V.kicad_sch (KiCad schematic)
At the start: 33 parts

Commit message: silkscreen and one part footprint and part number change for C3, C10, C15 and C22
Parts:
- C10, C3: footprint Capacitor_SMD:C_0201_0603Metric -> Capacitor_SMD:C_0603_1608Metric; Manufacturer Part Number C0603C473K3RACTU -> CL10B473KO8NNNC; Vendor Part Number 399-C0603C473K3RACTUCT-ND -> 1276-2079-1-ND
Changed lines of the file:
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@@
 			)
 		)
-		(property "Footprint" "Capacitor_SMD:C_0201_0603Metric"
+		(property "Footprint" "Capacitor_SMD:C_0603_1608Metric"
 			(at 230.8352 129.54 0)
 			(hide yes)
@@
 			)
 		)
-		(property "Datasheet" "https://www.yageogroup.com/content/datasheet/asset/file/KEM_C1002_X7R_SMD"
+		(property "Datasheet" "https://mm.digikey.com/Volume0/opasdata/d220001/medias/docus/658/CL10B473KO8NNNC_Spec.pdf"
 			(at 229.87 125.73 0)
 			(hide yes)
@@
 			)
 		)
-		(property "Description" "0.047 µF ±10% 25V Ceramic Capacitor X7R 0603 (1608 Metric)"
+		(property "Description" "0.047 µF ±10% 16V Ceramic Capacitor X7R 0603 (1608 Metric)"
 			(at 229.87 125.73 0)
 			(hide yes)
@@
 			)
 		)
-		(property "Manufacturer Part Number" "C0603C473K3RACTU"
+		(property "Manufacturer Part Number" "CL10B473KO8NNNC"
 			(at 229.87 125.73 0)
 			(hide yes)
@@
 			)
 		)
-		(property "Vendor Part Number" "399-C0603C473K3RACTUCT-ND"
+		(property "Vendor Part Number" "1276-2079-1-ND"
 			(at 229.87 125.73 0)
 			(hide yes)
@@
 			)
 		)
-		(property "Footprint" "Capacitor_SMD:C_0201_0603Metric"
+		(property "Footprint" "Capacitor_SMD:C_0603_1608Metric"
 			(at 65.7352 123.19 0)
 			(hide yes)
@@
 			)
 		)
-		(property "Datasheet" "https://www.yageogroup.com/content/datasheet/asset/file/KEM_C1002_X7R_SMD"
+		(property "Datasheet" "https://mm.digikey.com/Volume0/opasdata/d220001/medias/docus/658/CL10B473KO8NNNC_Spec.pdf"
 			(at 64.77 119.38 0)
 			(hide yes)
@@
 			)
 		)
-		(property "Description" "0.047 µF ±10% 25V Ceramic Capacitor X7R 0603 (1608 Metric)"
+		(property "Description" "0.047 µF ±10% 16V Ceramic Capacitor X7R 0603 (1608 Metric)"
 			(at 64.77 119.38 0)
 			(hide yes)
@@
 			)
 		)
-		(property "Manufacturer Part Number" "C0603C473K3RACTU"
+		(property "Manufacturer Part Number" "CL10B473KO8NNNC"
 			(at 64.77 119.38 0)
 			(hide yes)
@@
 			)
 		)
-		(property "Vendor Part Number" "399-C0603C473K3RACTUCT-ND"
+		(property "Vendor Part Number" "1276-2079-1-ND"
 			(at 64.77 119.38 0)
 			(hide yes)
